Commit message: fix(a2z1): apply 3-lens adversarial-review findings (2 blockers + geometry parity leg)
BLOCKER 1 (URDF): raw STLs were placed with COMPILED geom origins — MuJoCo
canonicalizes mesh assets (recenter/reorient, inverse baked into geom_pos/quat),
so every arm mesh visual + the 11 gripper collision hulls sat ~14 cm / ~136°
off. The generator now composes the canonicalization back in and NUMERICALLY
verifies its own composition per mesh (centroid + rotated-extent check vs the
raw STL vertex set); a new parity GEOMETRY leg pushes raw-vertex samples
through the WRITTEN URDF origins — 20/20 mesh placements now match MuJoCo
exactly. Also: mjGEOM constants fixed (6 is BOX, not sphere — the 4 gripper
contact pads were spheres of r=14mm instead of 8mm-thick boxes; box branch
added), mount euler now routed through a quaternion (MJCF intrinsic-xyz vs
URDF fixed-XYZ would silently desync a future non-trivial mount rotation),
sha-based mesh staleness.

BLOCKER 2 (env): IsaacLab joint position TARGETS are written only by action
terms (pinned to the 12 legs), so the arm's kp-1000 servos drove from stow to
the ALL-ZERO pose (ON joint2/joint3 limits) at episode start — "servo-held at
stow" did not exist train-side. New hold_arm_position_targets reset event
(ordered after the pose jitter) writes the arm targets to the jittered pose.

Also per review: arm actuators DCMotor → ImplicitActuatorCfg (menagerie servo
is a FLAT clip; DCMotor's torque-speed derating trained a weaker transient
hold than deploy — zero forward torque at |v|≥π), friction left unset so the
URDF-converted frictionloss survives import, gripper stow 0.0 → −0.1 (0.0 sat
ON the hard limit, outside soft limits — construction-error epsilon). Tests
extended to 52 checks (pad boxes, Implicit groups, target-hold ordering).

Co-Authored-By: Claude Fable 5 <noreply@anthropic.com>

File: resources/a2/urdf/a2z1.urdf (robot description, URDF)
Before this commit: robot a2, 31 links, 30 joints
Links:
- link z1_gripperMover: geometry collision box size=0.028 0.03 0.008; collision box size=0.028 0.03 0.008
- link z1_link06: geometry collision box size=0.028 0.03 0.008; collision box size=0.028 0.03 0.008
Joints:
- joint z1_mount_joint: origin xyz=-0.1 0 0.117 rpy=0 0 0 -> xyz=-0.1 0 0.117 rpy=0 -0 0
